Commit message: some changes to cost calcualiton: parameter changes

File: src/mircronrobot/turtlebot3/turtlebot3_description/urdf/turtlebot3_burger3.urdf.xacro (robot description, xacro)
@@ -143,17 +143,17 @@
   <xacro:include filename="$(find realsense2_description)/urdf/_d435.urdf.xacro"/>
   <sensor_d435 name="front_realsense" topics_ns="front_realsense" parent="base_link">
-    <origin xyz="0.032 0 0.5" rpy="0 0 0"/>
+    <origin xyz="0.032 0 0.5" rpy="0 -0.349 0"/>
   </sensor_d435>
    <xacro:include filename="$(find realsense2_description)/urdf/_d435.urdf.xacro"/>
   <sensor_d435 name="right_realsense" topics_ns="right_realsense" parent="base_link">
-    <origin xyz="-0.04 0.08 0.5" rpy="0 0 1.57"/>
+    <origin xyz="-0.04 0.08 0.5" rpy="0 -0.349 1.57"/>
   </sensor_d435>
   <xacro:include filename="$(find realsense2_description)/urdf/_d435.urdf.xacro"/>
   <sensor_d435 name="left_realsense" topics_ns="left_realsense" parent="base_link">
-    <origin xyz="-0.04 -0.08 0.5" rpy="0 0 -1.57"/>
+    <origin xyz="-0.04 -0.08 0.5" rpy="0 -0.349 -1.57"/>
   </sensor_d435>
   <xacro:include filename="$(find realsense2_description)/urdf/_d435.urdf.xacro"/>
   <sensor_d435 name="back_realsense" topics_ns="back_realsense" parent="base_link">
-    <origin xyz="-0.1 0 0.5" rpy="0 0 -3.14"/>
+    <origin xyz="-0.1 0 0.5" rpy="0 -0.349 -3.14"/>
   </sensor_d435>
  <!-- ULTRASONIC_SENSOR -->
